File: hardware/marine_gps.kicad_pcb (KiCad board)
At the start: 2 copper layers, 160 x 100 mm, 115 parts, among them CON101 GPIO1, CON102 GPIO3, P101 CONN_02X04, P102 CONN_02X02, P103 CONN_01X04, P104 CONN_01X11, P105 CONN_01X02, P106 CONN_01X06, P107 CONN_01X19, P108 CONN_01X01, P109 CONN_01X05, P110 CONN_01X03, P111 CONN_01X02, P112 CONN_01X05, P113 HE10-10, P114 CONN_01X03, P201 CONN_01X02, P301 CONN_02X03, P304 CONN_02X03, P305 CONN_02X02, P307 CONN_01X01, P308 CONN_01X03, P309 CONN_01X02, P310 CONN_01X03, P311 CONN_01X02, P401 HE10-10, P501 CONN_01X02, Q201 BC547, Q401 BSS138, Q501 BSS138, Q502 BSS138, Q503 DMG2307L, SW301 PWR, U201 TDA8541, U301 MCP1703A, U302 TPS560200, U303 TPS54228, U304 PIC18F25K22, U401 74lv126, U402 74lv126, U403 MAX3488E, U501 MCP2562, Y301 32.768Khz

Commit message: Swap D and S of Q503 (oups)
Parts:
- moved P501 7.63 mm to (117.5, 116.8)
- moved R502 4.18 mm to (120.0, 111.1), turned to 0 degrees
Connections:
- Q503 pad 2: Net-(P501-Pad1) -> +12V
- Q503 pad 3: +12V -> Net-(P501-Pad1)
Routing:
- net Net-(P501-Pad1): track 3.99 -> 24.1 mm
- net +12V: track 270.8 -> 289.2 mm
- net GND: track 858.4 -> 848.0 mm
- net /Marine GPS CAN/CAN_+12V: track 15.3 -> 7.14 mm
- net Net-(Q502-Pad3): track 19.6 -> 18.8 mm
