File: hardware/marine_gps_can.sch (KiCad schematic (older format))
At the start: 9 parts, among them P501 CONN_01X02, Q501 BSS138, Q502 BSS138, Q503 DMG2307L, U501 MCP2562

Commit message: Rename machine_gps_can to marine_gps_can (typo)
Parts:
- removed Q503: DMG2307L, TO_SOT_Packages_SMD:SOT-23, symbol Q_PMOS_GDS
- added Q503: DMG2307L, TO_SOT_Packages_SMD:SOT-23, symbol Q_PMOS_GSD
Connections:
- net +12V: now also Q503.2 (S)
- net at Q502.3 (D), R502.2: now also Q503.1 (G)
- net at P501.1 (P1): now also Q503.3 (D)
Changed lines of the file:
@@
 encoding utf-8
 Sheet 5 5
-Title ""
-Date ""
-Rev ""
-Comp ""
+Title "Marine GPS"
+Date "2016-03-19"
+Rev "1.1"
+Comp "Manuel Bouyer"
 Comment1 ""
 Comment2 ""
@@
 $Comp
 L MCP2562 U501
-U 1 1 56C61ED7
+U 1 1 00000000
 P 4400 2600
 F 0 "U501" H 4000 3050 50  0000 L BNN
@@
 $Comp
 L C_Small C501
-U 1 1 56C61ED8
+U 1 1 00000000
 P 2600 2600
 F 0 "C501" H 2610 2670 50  0000 L CNN
@@
 $Comp
 L C_Small C502
-U 1 1 56C61ED9
+U 1 1 00000000
 P 2850 2800
 F 0 "C502" H 2860 2870 50  0000 L CNN
@@
 $EndComp
 $Comp
-L Q_PMOS_GDS Q503
-U 1 1 56C61EDA
+L Q_PMOS_GSD Q503
+U 1 1 00000000
 P 5150 1850
 F 0 "Q503" H 5450 1900 50  0000 R CNN
@@
 F 2 "TO_SOT_Packages_SMD:SOT-23" H 5350 1950 50  0001 C CNN
 F 3 "" H 5150 1850 50  0000 C CNN
-F 4 "" H 5150 2450 60  0001 C CNN "P/N"
 	1    5150 1850
 	0    1    -1   0
@@
 $Comp
 L CONN_01X02 P501
-U 1 1 56C61EDB
+U 1 1 00000000
 P 5550 1550
 F 0 "P501" H 5550 1700 50  0000 C CNN
@@
 $Comp
 L R_Small R502
-U 1 1 56C61EDC
+U 1 1 00000000
 P 4850 1900
 F 0 "R502" H 4880 1920 50  0000 L CNN
@@
 $Comp
 L BSS138 Q501
-U 1 1 56C61EDD
+U 1 1 00000000
 P 3700 3600
 F 0 "Q501" H 3900 3675 50  0000 L CNN
@@
 $Comp
 L BSS138 Q502
-U 1 1 56C61EDE
+U 1 1 00000000
 P 5050 3600
 F 0 "Q502" H 5250 3675 50  0000 L CNN
@@
 $Comp
 L R_Small R501
-U 1 1 56C61EDF
+U 1 1 00000000
 P 3650 3900
 F 0 "R501" H 3680 3920 50  0000 L CNN
